File: SensibleRAM.kicad_pcb (KiCad board)
At the start: 2 copper layers, 42 x 55 mm, 5 parts, among them U1 MOS6561_socket, U2 MOS6561, U3 SN74LVC1G27DBVR, U4 SN74LVC1G10DBVR, U5 CY62256-70PC

Commit message: Moved init code to $1200 Fixed missing connection on PCB Added note about incomplete decoding to README
Routing:
- net MSel: track 38.3 -> 42.9 mm
